Commit message: adds kinect, etc

File: ardupilot_sitl_gazebo_plugin/urdf/erlecopter.xacro (robot description, xacro)
@@ -166,5 +166,5 @@
     ray_count_vertical="1"
     sensor_mesh="lidar_lite_v2_withRay/meshes/lidar_lite_v2_withRay.dae">
-    <origin xyz="0.13 0.0 0.02" rpy="0 0 0"/>
+    <origin xyz="0.13 0.0 0.05" rpy="0 0 0"/>
   </xacro:lidar_sensor>
   <!-- Downward facing camera -->
@@ -198,4 +198,17 @@
     <origin xyz="0.17 0.0 0.0" rpy="0 0 0"/>
   </xacro:generic_camera>
+  <!-- Kinect camera -->
+  <xacro:include filename="$(find ardupilot_sitl_gazebo_plugin)/urdf/sensors/kinect.urdf.xacro" />
+  <xacro:sensor_kinect parent="base_link" radius_rotor="${radius_rotor}" />
+  <!-- Contact sensor -->
+<!--   <xacro:include filename="$(find ardupilot_sitl_gazebo_plugin)/urdf/sensors/contact.urdf.xacro" />
+  <xacro:sensor_contact
+    name="erlecopter/contact"
+    parent="base_link"
+    body_length="${body_length}"
+    body_width="${body_width}"
+    body_height="${body_height}">
+    <origin xyz="0.0 0.0 0.0" rpy="0 0 0"/>
+  </xacro:sensor_contact> -->
   <!-- Instantiate rotors -->
   <xacro:vertical_rotor
@@ -216,5 +229,5 @@
     mesh="erlecopter_prop"
     mesh_scale="${mesh_scale_prop}"
-    color="Yellow">
+    color="Red">
     <origin xyz="${arm_length_front_x} -${arm_length_front_y} ${rotor_offset_top}" rpy="0 0 0" />
     <xacro:insert_block name="rotor_inertia" />
@@ -257,5 +270,5 @@
     mesh="erlecopter_prop"
     mesh_scale="${mesh_scale_prop}"
-    color="Yellow">
+    color="Red">
     <origin xyz="${arm_length_front_x} ${arm_length_front_y} ${rotor_offset_top}" rpy="0 0 0" />
     <xacro:insert_block name="rotor_inertia" />

File: ardupilot_sitl_gazebo_plugin/urdf/sensors/generic_camera.urdf.xacro (robot description, xacro)
@@ -14,5 +14,5 @@
       <link name="${name}_link">
         <inertial>
-          <mass value="0.001" />
+          <mass value="0.0005" />
           <origin xyz="0 0 0" rpy="0 0 0" />
           <inertia ixx="0.0001" ixy="0" ixz="0" iyy="0.0001" iyz="0" izz="0.0001" />
@@ -42,5 +42,5 @@
     <link name="ardrone_base_${name}cam">
       <inertial>
-        <mass value="0.01" />
+        <mass value="0.005" />
         <origin xyz="0 0 0" />
         <inertia ixx="0.001"  ixy="0.0"  ixz="0.0"

File: ardupilot_sitl_gazebo_plugin/urdf/sensors/kinect.urdf.xacro (robot description, xacro)
@@ -1,13 +1,13 @@
 <?xml version="1.0"?>
 <robot name="sensor_kinect" xmlns:xacro="http://ros.org/wiki/xacro">
-  <property name="cam_px" value="1.63" />
-  <xacro:property name="kinect_cam_py" value="-0.0125"/>
-  <property name="cam_pz" value="0.68" />
+  <property name="cam_px" value="0.17" />
+  <xacro:property name="kinect_cam_py" value="0"/>
+  <property name="cam_pz" value="0.05" />
   <property name="cam_or" value="0" />
-  <property name="cam_op" value="0" />
+  <property name="cam_op" value="-0.2" />
   <property name="cam_oy" value="0" />
   <xacro:property name="M_PI" value="3.1415926535897931" />
   <!-- Parameterised in part by the values in turtlebot_properties.urdf.xacro -->
-  <xacro:macro name="sensor_kinect" params="parent">
+  <xacro:macro name="sensor_kinect" params="parent radius_rotor">
     <joint name="camera_rgb_joint" type="fixed">
       <origin xyz="${cam_px} ${kinect_cam_py} ${cam_pz}" rpy="${cam_or} ${cam_op} ${cam_oy}"/>
@@ -34,16 +34,16 @@
         </geometry>
       </visual>
-  	  <collision>
+  	  <!-- <collision>
         <origin xyz="0.0 0.0 0.0" rpy="0 0 0"/>
   	    <geometry>
   	      <box size="0.07271 0.27794 0.073"/>
   	    </geometry>
-  	  </collision>
+  	  </collision> -->
       <inertial>
-        <mass value="0.564" />
+        <mass value="0.005" />
         <origin xyz="0 0 0" />
-        <inertia ixx="0.003881243" ixy="0.0" ixz="0.0"
-                 iyy="0.000498940" iyz="0.0"
-                 izz="0.003879257" />
+        <inertia ixx="0.001"  ixy="0.0"  ixz="0.0"
+                 iyy="0.001"  iyz="0.0"
+                 izz="0.001" />
       </inertial>
     </link>
@@ -69,5 +69,5 @@
       <update_rate>20.0</update_rate>
       <camera>
-        <horizontal_fov>${60.0*M_PI/180.0}</horizontal_fov>
+        <horizontal_fov>${90.0*M_PI/180.0}</horizontal_fov>
         <image>
           <format>R8G8B8</format>
@@ -76,7 +76,15 @@
         </image>
         <clip>
-          <near>0.05</near>
-          <far>8.0</far>
+          <near>${1.1 * radius_rotor}</near>
+          <far>100.0</far>
         </clip>
+        <noise>
+          <type>gaussian</type>
+          <!-- Noise is sampled independently per pixel on each frame.
+               That pixel's noise value is added to each of its color
+               channels, which at that point lie in the range [0,1]. -->
+          <mean>0.0</mean>
+          <stddev>0.007</stddev>
+        </noise>
       </camera>
       <plugin name="kinect_camera_controller" filename="libgazebo_ros_openni_kinect.so">
